File: PreAMP_CIRCUIT/PreampCircuit/PreampCircuit.kicad_sch (KiCad schematic)
At the start: 7 parts, among them Q1 NJFET

Commit message: PREAMP CIRCUIT
SOURCE: https://www.homemade-circuits.com/diy-contact-mic-circuit/
Parts:
- added J1: AudioJack2, symbol Connector_Audio:AudioJack2
Connections:
- net GND: now also J1.S
- net at C1.2, R4.1: now also J1.T
Other:
- note added: "INPUT"
- note added: "OUTPUT"
- moved on the sheet: R4
Changed lines of the file:
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@@
 	(generator_version "9.0")
 	(paper "A5")
+	(text "OUTPUT"
+		(exclude_from_sim no)
+		(at 154.686 27.686 0)
+		(effects
+			(font
+				(size 1.27 1.27)
+			)
+		)
+	)
+	(text "INPUT"
+		(exclude_from_sim no)
+		(at 42.926 46.99 0)
+		(effects
+			(font
+				(size 1.27 1.27)
+			)
+		)
+	)
 	(junction
-		(at 121.92 19.05)
+		(at 105.41 66.04)
+		(diameter 0)
+		(color 0 0 0 0)
+	)
+	(junction
+		(at 121.92 21.59)
 		(diameter 0)
 		(color 0 0 0 0)
@@
 	)
 	(junction
-		(at 109.22 66.04)
-		(diameter 0)
-		(color 0 0 0 0)
-	)
-	(junction
 		(at 80.01 66.04)
 		(diameter 0)
@@
 	)
 	(junction
+		(at 105.41 35.56)
+		(diameter 0)
+		(color 0 0 0 0)
+	)
+	(junction
 		(at 121.92 66.04)
 		(diameter 0)
@@
 		(color 0 0 0 0)
 	)
-	(junction
-		(at 109.22 35.56)
-		(diameter 0)
-		(color 0 0 0 0)
-	)
 	(wire
 		(pts
@@
 	(wire
 		(pts
-			(xy 109.22 66.04) (xy 121.92 66.04)
-		)
-		(stroke
-			(width 0)
-			(type default)
-		)
-	)
-	(wire
-		(pts
-			(xy 138.43 66.04) (xy 138.43 40.64)
+			(xy 138.43 66.04) (xy 138.43 38.1)
 		)
 		(stroke
@@
 	(wire
 		(pts
-			(xy 121.92 45.72) (xy 121.92 19.05)
+			(xy 121.92 45.72) (xy 121.92 21.59)
+		)
+		(stroke
+			(width 0)
+			(type default)
+		)
+	)
+	(wire
+		(pts
+			(xy 121.92 21.59) (xy 121.92 19.05)
 		)
 		(stroke
@@
 	(wire
 		(pts
+			(xy 105.41 66.04) (xy 121.92 66.04)
+		)
+		(stroke
+			(width 0)
+			(type default)
+		)
+	)
+	(wire
+		(pts
 			(xy 66.04 43.18) (xy 72.39 43.18)
 		)
@@
 	(wire
 		(pts
-			(xy 138.43 40.64) (xy 142.24 40.64)
-		)
-		(stroke
-			(width 0)
-			(type default)
-		)
-	)
-	(wire
-		(pts
-			(xy 80.01 19.05) (xy 121.92 19.05)
+			(xy 138.43 38.1) (xy 158.75 38.1)
+		)
+		(stroke
+			(width 0)
+			(type default)
+		)
+	)
+	(wire
+		(pts
+			(xy 105.41 35.56) (xy 158.75 35.56)
+		)
+		(stroke
+			(width 0)
+			(type default)
+		)
+	)
+	(wire
+		(pts
+			(xy 80.01 21.59) (xy 121.92 21.59)
 		)
 		(stroke
@@
 	(wire
 		(pts
-			(xy 99.06 35.56) (xy 109.22 35.56)
-		)
-		(stroke
-			(width 0)
-			(type default)
-		)
-	)
-	(wire
-		(pts
-			(xy 109.22 53.34) (xy 109.22 66.04)
-		)
-		(stroke
-			(width 0)
-			(type default)
-		)
-	)
-	(wire
-		(pts
-			(xy 80.01 25.4) (xy 80.01 19.05)
-		)
-		(stroke
-			(width 0)
-			(type default)
-		)
-	)
-	(wire
-		(pts
-			(xy 109.22 35.56) (xy 142.24 35.56)
-		)
-		(stroke
-			(width 0)
-			(type default)
-		)
-	)
-	(wire
-		(pts
-			(xy 109.22 35.56) (xy 109.22 45.72)
+			(xy 99.06 35.56) (xy 105.41 35.56)
+		)
+		(stroke
+			(width 0)
+			(type default)
+		)
+	)
+	(wire
+		(pts
+			(xy 105.41 53.34) (xy 105.41 66.04)
+		)
+		(stroke
+			(width 0)
+			(type default)
+		)
+	)
+	(wire
+		(pts
+			(xy 80.01 25.4) (xy 80.01 21.59)
+		)
+		(stroke
+			(width 0)
+			(type default)
+		)
+	)
+	(wire
+		(pts
+			(xy 105.41 35.56) (xy 105.41 45.72)
 		)
 		(stroke
@@
 	(wire
 		(pts
-			(xy 80.01 66.04) (xy 109.22 66.04)
+			(xy 80.01 66.04) (xy 105.41 66.04)
 		)
 		(stroke
@@
 	(symbol
 		(lib_id "Device:R")
-		(at 109.22 49.53 0)
+		(at 105.41 49.53 0)
 		(unit 1)
 		(exclude_from_sim no)
@@
 		(fields_autoplaced yes)
 		(property "Reference" "R4"
-			(at 111.76 48.2599 0)
+			(at 107.95 48.2599 0)
 			(effects
 				(font
@@
 		)
 		(property "Value" "220k"
-			(at 111.76 50.7999 0)
+			(at 107.95 50.7999 0)
 			(effects
 				(font
@@
 		)
 		(property "Footprint" ""
-			(at 107.442 49.53 90)
+			(at 103.632 49.53 90)
 			(effects
 				(font
@@
 		)
 		(property "Datasheet" "~"
-			(at 109.22 49.53 0)
+			(at 105.41 49.53 0)
 			(effects
 				(font
@@
 		)
 		(property "Description" "Resistor"
-			(at 109.22 49.53 0)
+			(at 105.41 49.53 0)
 			(effects
 				(font
@@
 					(unit 1)
 				)
+			)
+		)
+	)
+	(symbol
+		(lib_id "Connector_Audio:AudioJack2")
+		(at 163.83 35.56 180)
+		(unit 1)
+		(exclude_from_sim no)
+		(in_bom yes)
+		(on_board yes)
+		(dnp no)
+		(property "Reference" "J1"
+			(at 164.465 44.45 0)
+			(effects
+				(font
+					(size 1.27 1.27)
+				)
+			)
+		)
+		(property "Value" "AudioJack2"
+			(at 164.465 41.91 0)
+			(effects
+				(font
+					(size 1.27 1.27)
+				)
+			)
+		)
+		(property "Footprint" ""
+			(at 163.83 35.56 0)
+			(effects
+				(font
+					(size 1.27 1.27)
+				)
+				(hide yes)
+			)
+		)
+		(property "Datasheet" "~"
+			(at 163.83 35.56 0)
+			(effects
+				(font
+					(size 1.27 1.27)
+				)
+				(hide yes)
+			)
+		)
+		(property "Description" "Audio Jack, 2 Poles (Mono / TS)"
+			(at 163.83 35.56 0)
+			(effects
+				(font
+					(size 1.27 1.27)
+				)
+				(hide yes)
+			)
+		)
+		(pin "T"
+		)
+		(pin "S"
+		)
+		(instances
+			(project ""
+				(path "/2bfd962c-74c5-4142-b55e-dbdb00ee74c3"
+					(reference "J1")
+					(unit 1)
+				)
