File: PreAMP_CIRCUIT/PreampCircuit/PreampCircuit.kicad_sch (KiCad schematic)
At the start: 11 parts, among them J1 AudioJack2, J2 Conn_01x02_Pin, Q2 2N3819

Commit message: ROUTING
Parts:
- removed RV1: R_Pot 3M, Potentiometer_SMD:Potentiometer_Bourns_3314G_Vertical, symbol Device:R_Potentiometer
- added R1: PTN16-A10220K1B1, pot:POT_PTN16-A10220K1B1, symbol pot:PTN16-A10220K1B1
- BT1: footprint Connector_PinSocket_2.00mm:PinSocket_1x02_P2.00mm_Vertical_SMD_Pin1Right -> 2pads:2pads
- J1: footprint (none) -> 2pads:2pads
- J2: footprint Connector_PinSocket_2.00mm:PinSocket_1x02_P2.00mm_Vertical_SMD_Pin1Right -> 2pads
Connections:
- net GND: now also R1.3
- net at R5.2: now also R1.2
Other:
- moved on the sheet: BT1, C1, C2, J1, J2, Q2, R2, R3, R4, R5
